File: hw/pcb/atmt.sch (EAGLE design)
At the start: 39 parts, among them IC1 LP2989IM-3.3_NOPB, IC2 ESP32-WROOM-32UE_M113EH6400UH3, IC3 L293DD

Commit message: first commit of control-sysetm
Parts:
- removed C1: 22uF, SparkFun-Passives:CAP0805
- added C11: 22u, rcl:CPOL-USE2-5
- added D2: 1N4148W-7-F, SamacSys_Parts:1N4148W-7-F
Connections:
- net 3V3: now also C11.+, D2.A; no longer C1.1
- net 4.5V: now also D2.K
- net ECHO2: now also IC2.IO35; no longer IC2.IO16
- net GND: now also C11.-; no longer C1.2
- net TRIG1: now also IC2.IO16; no longer IC2.IO35
Other:
- moved on the sheet: R1
