File: hw/pcb/atmt.brd (EAGLE design)
At the start: 63 x 57 mm, 39 parts, among them IC1 LP2989IM-3.3_NOPB, IC2 ESP32-WROOM-32UE_M113EH6400UH3, IC3 L293DD

Commit message: first commit of control-sysetm
Parts:
- removed C1: 22uF, SparkFun-Passives:0805
- added C11: 22u, rcl:E2-5
- added D2: 1N4148W-7-F, SamacSys_Parts:SOD3716X115N
- moved R4 79.7 mm to (52.7, 36.7), turned to 270 degrees
- moved JP20 75.2 mm to (55.9, 35.5), flipped to the bottom, turned to 90 degrees
- moved R3 73.1 mm to (45.8, 37.4)
- moved JP19 68.6 mm to (49.3, 38.2), flipped to the bottom, turned to 90 degrees
- moved C2 2.82 mm to (40.5, 14.6)
- moved JP1 2.28 mm to (9.70, 51.6), flipped to the bottom, turned to 270 degrees
- moved R2 0.99 mm to (34.7, 12.6)
- moved C3 0.94 mm to (34.5, 15.1)
- moved JP2 0.92 mm to (46.1, 44.9), flipped to the bottom, turned to 90 degrees
Connections:
- net 3V3: now also C11.+, D2.2; no longer C1.1
- net 4.5V: now also D2.1
- net ECHO2: now also IC2.7; no longer IC2.27
- net GND: now also C11.-; no longer C1.2
- net TRIG1: now also IC2.27; no longer IC2.7
Routing:
- net 3V3: track 165.4 -> 226.7 mm
- net GND: track 176.6 -> 200.3 mm
- net M1_2: track 13.9 -> 23.4 mm
- net M2_2: track 11.0 -> 20.4 mm
- net TRIG1: track 26.5 -> 35.2 mm, vias 0 -> 1
- net 4.5V: track 193.6 -> 200.4 mm
- net N$3: track 0.00 -> 4.59 mm
- net N$2: track 0.00 -> 2.79 mm
- net ECHO2: track 44.7 -> 42.0 mm, vias 1 -> 2
- net M1_1: track 12.3 -> 10.8 mm
- net M2_1: track 7.98 -> 9.48 mm
- net M2F: track 47.0 -> 46.5 mm
Other:
- board text added: "+3V3"
- board text added: "+4V5"

Commit message: new board and some code..
Routing:
- net 3V3: track 226.7 -> 222.4 mm
- net TX: track 37.1 -> 38.0 mm
- net 4.5V: track 200.4 -> 199.7 mm
- net M1F: track 29.7 -> 29.1 mm
Other:
- board text added: "A T M T Pär Sundbäck Version 2.0 2021-03-01"
- board text removed: "A T M T Pär Sundbäck Version 2.0 2021-02-15"
