File: hw/pcb-kicad/atmt-kcad/atmt-kcad.kicad_sch (KiCad schematic)
At the start: 14 parts, among them J3 Conn_01x04_Male, J4 Conn_01x04_Male, U1 ESP32-WROOM-32U, U2 LP2987-3.3_SOIC8_VSSOP8, U3 4504, U4 L293

Commit message: Before refactoring
Parts:
- removed C2: C_Polarized, Capacitor_THT:CP_Axial_L11.0mm_D6.0mm_P18.00mm_Horizontal, symbol Device:C_Polarized
- removed U4: L293, Package_DIP:DIP-16_W7.62mm_SMDSocket_SmallPads, symbol Driver_Motor:L293
- added C2, C7: 100n, Capacitor_SMD:C_0805_2012Metric_Pad1.18x1.45mm_HandSolder, symbol Device:C
- added D2: PowerOn, LED_THT:LED_D3.0mm, symbol Device:LED
- added J1: Reset, Connector_PinHeader_2.54mm:PinHeader_1x02_P2.54mm_Vertical, symbol Connector:Conn_01x02_Pin
- added J10: JTAG, Connector_PinHeader_2.54mm:PinHeader_1x04_P2.54mm_Vertical, symbol Connector:Conn_01x04_Pin
- added J11: BAT+, Connector_Wire:SolderWire-1.5sqmm_1x01_D1.7mm_OD3mm, symbol Connector:Conn_01x01_Pin
- added J12: BAT-, Connector_Wire:SolderWire-1.5sqmm_1x01_D1.7mm_OD3mm, symbol Connector:Conn_01x01_Pin
- added J13: Steering, Connector_Phoenix_MSTB:PhoenixContact_MSTBA_2,5_2-G-5,08_1x02_P5.08mm_Horizontal, symbol Connector:Conn_01x02_Pin
- added J14: Motor, Connector_Phoenix_MSTB:PhoenixContact_MSTBA_2,5_2-G-5,08_1x02_P5.08mm_Horizontal, symbol Connector:Conn_01x02_Pin
- added J15: BOOT, Connector_PinHeader_2.54mm:PinHeader_1x02_P2.54mm_Vertical, symbol Connector:Conn_01x02_Pin
- added J16: Light, Connector_PinHeader_2.54mm:PinHeader_1x03_P2.54mm_Vertical, symbol Connector:Conn_01x03_Pin
- added J17: Buck/Boost, Connector_PinHeader_2.54mm:PinHeader_1x03_P2.54mm_Vertical, symbol Connector:Conn_01x03_Pin
- added J2: PowerSw, Connector_PinHeader_2.54mm:PinHeader_1x02_P2.54mm_Vertical, symbol Connector:Conn_01x02_Pin
- added J5: US-Right, Connector_PinHeader_2.54mm:PinHeader_1x04_P2.54mm_Vertical, symbol Connector:Conn_01x04_Male
- added J6: US-Left, Connector_PinHeader_2.54mm:PinHeader_1x04_P2.54mm_Vertical, symbol Connector:Conn_01x04_Male
- added J7: I2Cx2, Connector_PinHeader_2.54mm:PinHeader_1x04_P2.54mm_Vertical, symbol Connector:Conn_01x04_Pin
- added J8: PRG, Connector_PinHeader_2.54mm:PinHeader_1x04_P2.54mm_Vertical, symbol Connector:Conn_01x04_Pin
- added J9: I2C_1, Connector_PinHeader_2.54mm:PinHeader_1x04_P2.54mm_Vertical, symbol Connector:Conn_01x04_Pin
- added R2, R5, R6: 10k, Resistor_SMD:R_0805_2012Metric_Pad1.20x1.40mm_HandSolder, symbol Device:R
- added R3: 470k, Resistor_SMD:R_0805_2012Metric_Pad1.20x1.40mm_HandSolder, symbol Device:R
- added R4: 100k, Resistor_SMD:R_0805_2012Metric_Pad1.20x1.40mm_HandSolder, symbol Device:R
- added R7: 470, Resistor_SMD:R_0805_2012Metric_Pad1.20x1.40mm_HandSolder, symbol Device:R
- added U4: L293DD, MyFootprints:SO-20_STM, symbol added:L293DD
- C1, C4: value C -> 10u
- C3: value C -> 100n
- C5: value C -> 1u
- C6: value C_Polarized -> 22u
- J3: value Conn_01x04_Male -> US-Front
- J4: value Conn_01x04_Male -> US-Rear
- R1: value R -> 330k
- U2: value LP2987-3.3_SOIC8_VSSOP8 -> LP2987-3.3
Connections:
- net 5V: now reaches U3.1 (VCC)
- net 5V: now also J3.1 (Pin_1), J4.1 (Pin_1), U3.13 (Select), J16.1 (Pin_1), J17.3 (Pin_3), J5.1 (Pin_1), J6.1 (Pin_1), U4.10 (VS)
- net Echo4L: now reaches U3.10 (Dout)
- net Echo4L: now also U1.30 (IO18)
- net 3V3: now reaches U3.16 (VDD)
- net 3V3: now also C3.1, C4.2, C6.1, D1.2 (A), R1.2, U1.2 (VDD), U2.5 (OUT), U2.6 (SENSE), J7.1 (Pin_1), J8.1 (Pin_1), J9.1 (Pin_1), R2.1, R5.1, R6.1, R7.2, U4.20 (VSS)
- net Echo1L: now reaches U3.2 (Aout)
- net Echo1L: now also U1.6 (IO34)
- net Echo1: now reaches U3.3 (Ain)
- net Echo1: now also J3.3 (Pin_3)
- net Echo2L: now reaches U3.4 (Bout)
- net Echo2L: now also U1.7 (IO35)
- net Echo2: now reaches U3.5 (Bin)
- net Echo2: now also J5.3 (Pin_3)
- net Echo3L: now reaches U3.6 (Cout)
- net Echo3L: now also U1.10 (IO25)
- net Echo3: now reaches U3.7 (Cin)
- net Echo3: now also J6.3 (Pin_3)
- net GND: now reaches U3.8 (VSS)
- net GND: now also C1.1, C3.2, C4.1, C5.2, C6.2, J3.4 (Pin_4), J4.4 (Pin_4), U1.1 (GND), U1.15 (GND), U1.38 (GND), U1.39 (GND), U2.3 (GND), C2.2, C7.2, D2.1 (K), J1.2 (Pin_2), J12.1 (Pin_1), J15.2 (Pin_2), J16.3 (Pin_3), J17.2 (Pin_2), J5.4 (Pin_4), J6.4 (Pin_4), J7.2 (Pin_2), J8.2 (Pin_2), J9.2 (Pin_2), R4.2, U4.14 (GND), U4.15 (GND), U4.16 (GND), U4.17 (GND), U4.4 (GND), U4.5 (GND), U4.6 (GND), U4.7 (GND)
- net Echo4: now reaches U3.9 (Din)
- net Echo4: now also J4.3 (Pin_3)
- net Trig4: now reaches J4.2 (Pin_2)
- net Trig4: now also U1.31 (IO19)
- net Trig1: now reaches J3.2 (Pin_2)
- net Trig1: now also U1.27 (IO16)
- net B+: now reaches U2.4 (IN)
- net B+: now also C1.2, J17.1 (Pin_1), J2.2 (Pin_2), R3.1
- net at U2.7 (~{ERROR}): now also R1.1
- net at U2.8 (~{SHTD}): now also D1.1 (K)
- net Trig3: now reaches U1.11 (IO26)
- net Trig3: now also J6.2 (Pin_2)
- net M2F: now reaches U1.12 (IO27)
- net M2F: now also U4.12 (INPUT_3)
- net TMS: now reaches U1.13 (IO14)
- net TMS: now also J10.1 (Pin_1)
- net TDI: now reaches U1.14 (IO12)
- net TDI: now also J10.2 (Pin_2)
- net TCK: now reaches U1.16 (IO13)
- net TCK: now also J10.3 (Pin_3)
- net TDO: now reaches U1.23 (IO15)
- net TDO: now also J10.4 (Pin_4)
- net M1E: now reaches U1.24 (IO2)
- net M1E: now also U4.1 (ENABLE_1)
- net IO0: now reaches U1.25 (IO0)
- net IO0: now also J15.1 (Pin_1)
- net M1F: now reaches U1.26 (IO4)
- net M1F: now also U4.2 (INPUT_1)
- net Trig2: now reaches U1.28 (IO17)
- net Trig2: now also J5.2 (Pin_2)
- net M1R: now reaches U1.29 (IO5)
- net M1R: now also U4.9 (INPUT_2)
- net EN: now reaches U1.3 (EN)
- net EN: now also C5.1, C2.1, J1.1 (Pin_1), R2.2
- net SDA: now reaches U1.33 (IO21)
- net SDA: now also J7.4 (Pin_4), J9.4 (Pin_4), R6.2
- net RX: now reaches U1.34 (RXD0/IO3)
- net RX: now also J8.3 (Pin_3)
- net TX: now reaches U1.35 (TXD0/IO1)
- net TX: now also J8.4 (Pin_4)
- net SCL: now reaches U1.36 (IO22)
- net SCL: now also J7.3 (Pin_3), J9.3 (Pin_3), R5.2
- net M2R: now reaches U1.37 (IO23)
- net M2R: now also U4.19 (INPUT_4)
- net L1: now reaches U1.8 (IO32)
- net L1: now also J16.2 (Pin_2)
- net M2E: now reaches U1.9 (IO33)
- net M2E: now also U4.11 (ENABLE_2)
- new net: J11.1 (Pin_1), J2.1 (Pin_1)
- new net: D2.2 (A), R7.1
- new net ADC: C7.1, R3.2, R4.1
- new net M1_1: J14.2 (Pin_2), U4.3 (OUTPUT_1)
- new net M1_2: J14.1 (Pin_1), U4.8 (OUTPUT_2)
- new net M2_1: J13.2 (Pin_2), U4.18 (OUTPUT_4)
- new net M2_2: J13.1 (Pin_1), U4.13 (OUTPUT_3)
Other:
- note added: "I2C"
- note added: "Light"
- note added: "Motor connections"
- note added: "Motor control"
- note added: "Power-supply"
- note added: "Programming and debug"
- note added: "Start and reset"
- note added: "Switchregulator step-up/step-down 5V 1A By replacing B+ <-> 5V with a wire the stable 5V becomes B+"
- note added: "Ultrasonic sensors"
- moved on the sheet: C1, C3, C4, C5, C6, D1, J3, J4, R1, U1, U2, U3

Commit message: added pin-descr
Connections:
- net ADC: now also U1.4 (SENSOR_VP)
Changed lines of the file:
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@@
+	(wire
+		(pts
+			(xy 199.39 91.44) (xy 207.01 91.44)
+		)
+		(stroke
+			(width 0)
+			(type default)
+		)
+	)
 	(wire
 		(pts
@@
 	(text "Motor control"
 		(exclude_from_sim no)
-		(at 347.726 140.97 0)
+		(at 341.884 137.922 0)
 		(effects
 			(font
@@
 	(text "Programming and debug"
 		(exclude_from_sim no)
-		(at 93.726 182.626 0)
+		(at 73.152 184.912 0)
 		(effects
 			(font
@@
 	(text "Power-supply"
 		(exclude_from_sim no)
-		(at 99.06 80.01 0)
+		(at 99.568 80.01 0)
 		(effects
 			(font
@@
 	(text "Ultrasonic sensors"
 		(exclude_from_sim no)
-		(at 104.14 272.542 0)
+		(at 116.84 258.572 0)
 		(effects
 			(font
@@
 		(fields_autoplaced yes)
 		(effects
+			(font
+				(size 1.27 1.27)
+			)
+			(justify left bottom)
+		)
+	)
+	(label "ADC"
+		(at 199.39 91.44 0)
+		(fields_autoplaced yes)
+		(effects

Commit message: New kicad and a new hello-world-sw
Parts:
- removed U2: LP2987-3.3, Package_SO:SOIC-8_3.9x4.9mm_P1.27mm, symbol Regulator_Linear:LP2987-3.3_SOIC8_VSSOP8
- added C8: 100n, Capacitor_SMD:C_0805_2012Metric_Pad1.18x1.45mm_HandSolder, symbol Device:C
- added U2: LP2988-3.3_SOIC8_VSSOP8, Package_SO:SOIC-8_3.9x4.9mm_P1.27mm, symbol Regulator_Linear:LP2988-3.3_SOIC8_VSSOP8
Connections:
- net 3V3: now also U2.5 (OUT), U2.6 (SENSE)
- net B+: now also D1.1 (K), U2.4 (IN), U2.8 (~{SHTD})
- net GND: now also C8.2, U2.3 (GND)
- net at R1.1: now also U2.7 (~{ERROR})
- new net: C8.1, U2.1 (BP)
